Commit message: first comm

File: catkin_ws/src/multi_robot_scenario/xacro/p3dx/pioneer3dx.xacro (robot description, xacro)
@@ -6,16 +6,11 @@
   <xacro:include filename="$(find multi_robot_scenario)/xacro/p3dx/pioneer3dx_body.xacro"/>
   <xacro:pioneer3dx_body name="chassis" parent="base_link" meshes="package://gazebo_plugins/test/multi_robot_scenario/meshes/p3dx"/>
-  <!-- Laser -->
-  <xacro:include filename="$(find multi_robot_scenario)/xacro/laser/hokuyo.xacro"/>
-  <xacro:laser name="front_laser" parent="chassis" xyz="0.125 0 0.25" rpy="0 0 0" meshes="package://gazebo_plugins/test/multi_robot_scenario/meshes/laser"/>
-  <!-- GPU Laser
-  <xacro:include filename="$(find multi_robot_scenario)/xacro/laser/hokuyo_gpu.xacro"/>
-  <xacro:laser_gpu name="front_laser" parent="chassis" xyz="0.16 0 0.1" rpy="0 0 0" meshes="package://gazebo_plugins/test/multi_robot_scenario/meshes/laser" />
-    -->
-  <xacro:include filename="$(find multi_robot_scenario)/xacro/camera/camera.xacro"/>
-  <xacro:cam name="front_camera" parent="chassis" xyz="0.025 0 0.32" rpy="0 0 0" />
-  <xacro:include filename="$(find multi_robot_scenario)/xacro/camera/cameraD.xacro"/>
-  <xacro:camD name="cameraD" parent="chassis" xyz="0.025 0 0.32" rpy="0 0 0" />
-  <!-- Velodyne -->
+  <!-- uncomment 13 to 29 the below line to use other sensors like velodyne and hokuyo camera -->
+  <!-- <xacro:include filename="$(find multi_robot_scenario)/xacro/laser/hokuyo.xacro"/>
+  <xacro:laser name="front_laser" parent="chassis" xyz="0.125 0 0.25" rpy="0 0 0" meshes="package://gazebo_plugins/test/multi_robot_scenario/meshes/laser"/> -->
+  <!-- <xacro:include filename="$(find multi_robot_scenario)/xacro/camera/camera.xacro"/>
+  <xacro:cam name="front_camera" parent="chassis" xyz="0.025 0 0.32" rpy="0 0 0" /> -->
+  <!-- <xacro:include filename="$(find multi_robot_scenario)/xacro/camera/cameraD.xacro"/>
+  <xacro:camD name="cameraD" parent="chassis" xyz="0.025 0 0.32" rpy="0 0 0" /> -->
   <xacro:include filename="$(find velodyne_description)/urdf/VLP-16.urdf.xacro"/>
   <xacro:VLP-16 parent="base_link" name="velodyne" topic="/velodyne_points" hz="10" samples="360" gpu="false" min_angle="-1.57" max_angle="1.57" min_range="0.1">

File: catkin_ws/src/multi_robot_scenario/xacro/p3dx/pioneer3dx_body.xacro (robot description, xacro)
@@ -8,21 +8,28 @@
   <xacro:include filename="pioneer3dx_sonar.xacro"/>
   <xacro:include filename="pioneer3dx_plugins.xacro"/>
+  <xacro:include filename="$(find realsense2_description)/urdf/_d435.urdf.xacro"/>
   <xacro:macro name="pioneer3dx_body" params="name parent meshes">
     <!-- base_link -->
     <link name="${parent}"/>
     <!-- Chassis -->
-    <xacro:pioneer_chassis name="${name}" parent="base_link" xyz="0 0 0" rpy="0 0 0"  meshes="${meshes}"/>
+    <xacro:pioneer_chassis name="${name}" parent="base_link" xyz="0 0 0" rpy="0 0 0" meshes="${meshes}"/>
     <!-- Front Sonar -->
-    <xacro:pioneer_sonar name="sonar" parent="${name}" xyz="0.109 0 0.209" rpy="0 0 0"  meshes="${meshes}"/>
+    <xacro:pioneer_sonar name="sonar" parent="${name}" xyz="0.109 0 0.209" rpy="0 0 0" meshes="${meshes}"/>
     <!-- Akku0 -->
-    <xacro:battery_block name="battery0" parent="${name}" x="-0.14" y="0.00"  z="0.13" mass="2.5" />
+    <xacro:battery_block name="battery0" parent="${name}" x="-0.14" y="0.00" z="0.13" mass="2.5" />
     <!-- Wheels -->
-    <xacro:pioneer_wheel side="right" parent="${name}"  xyz="0  0.15 0.09" rpy="0 0 0" radius="0.09" meshes="${meshes}"/>
-    <xacro:pioneer_wheel side="left"  parent="${name}"  xyz="0 -0.15 0.09" rpy="0 0 0" radius="0.09" meshes="${meshes}"/>
-    <xacro:pioneer_swivel parent="${name}"  xyz="-0.185 0 0.055" rpy="0 0 0" meshes="${meshes}"/>
+    <xacro:pioneer_wheel side="right" parent="${name}" xyz="0  0.15 0.09" rpy="0 0 0" radius="0.09" meshes="${meshes}"/>
+    <xacro:pioneer_wheel side="left" parent="${name}" xyz="0 -0.15 0.09" rpy="0 0 0" radius="0.09" meshes="${meshes}"/>
+    <xacro:pioneer_swivel parent="${name}" xyz="-0.185 0 0.055" rpy="0 0 0" meshes="${meshes}"/>
     <!-- Motor plugin -->
     <xacro:pioneer3dx_diff_drive />
     <!-- Joints plugin -->
     <xacro:pioneer3dx_joints_state_publisher />
+    <!-- Prismatic plugin -->
+    <!-- <xacro:pioneer3dx_prisma />-->
+    <xacro:gazebo_control />
+    <xacro:sensor_d435 name="camera" topics_ns="realsense_camera" parent="base_link" publish_pointcloud="true">
+    <origin xyz="0.15 0 0.32" rpy="0 0 0" />
+  </xacro:sensor_d435>
   </xacro:macro>
 </robot>

File: catkin_ws/src/multi_robot_scenario/xacro/p3dx/pioneer3dx_plugins.xacro (robot description, xacro)
@@ -3,34 +3,38 @@
   <xacro:macro name="pioneer3dx_joints_state_publisher">
     <gazebo>
-        <plugin name="joint_state_publisher" filename="libgazebo_ros_joint_state_publisher.so">
-          <robotNamespace></robotNamespace>
-          <jointName>chassis_swivel_joint, swivel_wheel_joint, left_hub_joint, right_hub_joint</jointName>
-          <updateRate>50.0</updateRate>
-          <alwaysOn>true</alwaysOn>
-        </plugin>
+      <plugin name="joint_state_publisher" filename="libgazebo_ros_joint_state_publisher.so">
+        <robotNamespace></robotNamespace>
+        <jointName>chassis_swivel_joint, swivel_wheel_joint, left_hub_joint, right_hub_joint</jointName>
+        <updateRate>50.0</updateRate>
+        <alwaysOn>true</alwaysOn>
+      </plugin>
     </gazebo>
   </xacro:macro>
   <xacro:macro name="pioneer3dx_diff_drive">
     <gazebo>
-        <plugin name="differential_drive_controller" filename="libgazebo_ros_diff_drive.so">
-            <rosDebugLevel>Debug</rosDebugLevel>
-            <robotNamespace></robotNamespace>
-            <publishWheelTF>false</publishWheelTF>
-            <publishWheelJointState>true</publishWheelJointState>
-            <alwaysOn>true</alwaysOn>
-            <leftJoint>left_hub_joint</leftJoint>
-            <rightJoint>right_hub_joint</rightJoint>
-            <wheelSeparation>0.3</wheelSeparation>
-            <wheelDiameter>0.18</wheelDiameter>
-            <wheelTorque>20</wheelTorque>
-            <wheelAcceleration>1.8</wheelAcceleration>
-            <commandTopic>cmd_vel</commandTopic>
-            <odometryTopic>odom</odometryTopic>
-            <odometryFrame>odom</odometryFrame>
-            <odometrySource>world</odometrySource>
-            <robotBaseFrame>base_link</robotBaseFrame>
-	    <updateRate>50</updateRate>
-        </plugin>
+      <plugin name="differential_drive_controller" filename="libgazebo_ros_diff_drive.so">
+        <rosDebugLevel>Debug</rosDebugLevel>
+        <robotNamespace>r1</robotNamespace>
+        <publishWheelTF>false</publishWheelTF>
+        <publishWheelJointState>true</publishWheelJointState>
+        <alwaysOn>true</alwaysOn>
+        <leftJoint>left_hub_joint</leftJoint>
+        <rightJoint>right_hub_joint</rightJoint>
+        <wheelSeparation>0.3</wheelSeparation>
+        <wheelDiameter>0.18</wheelDiameter>
+        <wheelTorque>40</wheelTorque>
+        <!-- # settings to robot -->
+        <wheelAcceleration>2.2</wheelAcceleration>
+        <commandTopic>cmd_vel</commandTopic>
+        <odometryTopic>odom</odometryTopic>
+        <odometryFrame>odom</odometryFrame>
+        <odometrySource>world</odometrySource>
+        <robotBaseFrame>base_link</robotBaseFrame>
+        <updateRate>50</updateRate>
+      </plugin>
     </gazebo>
   </xacro:macro>
+<xacro:macro name="gazebo_control">
+<gazebo> <plugin name="gazebo_ros_control" filename="libgazebo_ros_control.so">   </plugin> </gazebo>
+</xacro:macro>
 </robot>
